File: PCB/Midiboard.kicad_sch (KiCad schematic)
At the start: 11 parts, among them J1 Capacitive_keys, SW1 SW_Push, SW2 SW_Push, SW3 SW_Push, SW4 RotaryEncoder_Switch_MP, U1 Waveshare ESP32-S3-ZERO

Commit message: Add files via upload
Parts:
- D1, D2, D3: LCSC Part # (none) -> C5149201
- J1: LCSC Part # (none) -> C2932700
- RV1, RV2: footprint Potentiometer_THT:Potentiometer_Bourns_PTA1543_Single_Slide -> Potentiometer_THT:Potentiometer_Bourns_PTA2043_Single_Slide; LCSC Part # (none) -> C5272874
- SW1, SW2, SW3: footprint Hackclub Footprints:Kailh Choc Low-Profile Switches -> Button_Switch_Keyboard:SW_Cherry_MX_1.00u_PCB
- SW4: LCSC Part # (none) -> C470754
- U1: LCSC (none) -> C9900190773
Connections:
- net ENC1_A: now also U1.5 (GP5); no longer U1.1 (GP1)
- net ENC1_B: now also U1.6 (GP6); no longer U1.2 (GP2)
- net LED: now also U1.4 (GP4); no longer U1.3 (GP3)
- net SWITCH1: now also U1.1 (GP1); no longer U1.4 (GP4)
- net SWITCH2: now also U1.2 (GP2); no longer U1.5 (GP5)
- net SWITCH3: now also U1.3 (GP3); no longer U1.6 (GP6)

Commit message: Add files via upload
Connections:
- net SLIDE1: now also U1.1 (GP1); no longer U1.TX
- net SLIDE2: now also U1.2 (GP2); no longer U1.RX
- net SWITCH1: now also U1.TX; no longer U1.1 (GP1)
- net SWITCH2: now also U1.RX; no longer U1.2 (GP2)
Changed lines of the file:
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@@
+		)
+	)
+	(label "SLIDE1"
+		(at 102.87 102.87 0)
+		(effects
+			(font
+				(size 1.27 1.27)
+			)
+			(justify left bottom)
 		)
 	)
@@
 		)
 	)
+	(label "SLIDE2"
+		(at 102.87 105.41 0)
+		(effects
+			(font
+				(size 1.27 1.27)
+			)
+			(justify left bottom)
+		)
+	)
 	(label "TOUCH3"
 		(at 167.64 104.14 0)
@@
 		)
 	)
+	(label "SWITCH1"
+		(at 102.87 97.79 0)
+		(effects
+			(font
+				(size 1.27 1.27)
+			)
+			(justify left bottom)
+		)
+	)
 	(label "TOUCH5"
 		(at 149.86 102.87 0)
@@
 		)
 	)
-	(label "SLIDE2"
+	(label "SWITCH2"
 		(at 102.87 95.25 0)
-		(effects
-			(font
-				(size 1.27 1.27)
-			)
-			(justify left bottom)
-		)
-	)
-	(label "SWITCH2"
-		(at 102.87 105.41 0)
 		(effects
 			(font
@@
 		(effects
 			(font
-				(size 1.27 1.27)
-			)
-			(justify left bottom)
-		)
-	)
-	(label "SLIDE1"
-		(at 102.87 97.79 0)
-		(effects
-			(font
-				(size 1.27 1.27)
-			)
-			(justify left bottom)
-		)
-	)
-	(label "SWITCH1"
-		(at 102.87 102.87 0)
-		(effects
-			(font
